File: electric/scheme-proto/clock-proto.sch (KiCad schematic (older format))
At the start: 40 parts

Commit message: Designing clock-proto.
Parts:
- added D? (x2): DIODESCH, ~, symbol DIODESCH
- added U?: NCP1402, ~, symbol NCP1402
Connections:
- net labels added: from-adapter, from-battery, power
- net labels removed: +5v
- wire segments 111 -> 118
Other:
- moved on the sheet: C?, Q?, R?, U?A, U?B

Commit message: Drawing scheme.
Parts:
- removed W?: short, symbol TEST
- added C? (x2): 4u7, ~, symbol C
- added C?: CP1, ~, symbol CP1
- added C? (x2): 100n, symbol C
- added C? (x2): 4u7, symbol C
- added C?: 2.2n, symbol C
- added C?: 1n, ~, symbol C
- added D?: 1N5819, ~, symbol DIODESCH
- added D?: 1N5819, symbol DIODESCH
- added L?: INDUCTOR, ~, symbol INDUCTOR
- added L?: INDUCTOR, symbol INDUCTOR
- added R?: 10k, symbol R
- added R?: 30k, symbol R
- added R? (x8): 0, ~, symbol R
- added R?: 10k, ~, symbol R
- added U?: NCP3063, symbol NCP3063
- D? (x2): value DIODESCH -> 1N5819
Connections:
- net labels added: 5v, boost-out, from-discovery-3.3v, from-discovery-5v, snd-amp-in, sound-dac, speaker-1, speaker-2
- net labels removed: filtered-pwm
- wire segments 118 -> 187
Other:
- moved on the sheet: C?, D?, Q?, R?, U?A, U?B

Commit message: Made circuit. Supposed to add a few LEDs to provide LCD back light
Parts:
- removed C? (x2): 4u7, ~, symbol C
- removed C?: CP1, ~, symbol CP1
- removed D?: 1N5819, ~, symbol DIODESCH
- removed L?: INDUCTOR, ~, symbol INDUCTOR
- removed R?: 0, ~, symbol R
- removed U?: NCP1402, ~, symbol NCP1402
- added C? (x3): 100n, symbol C
- added C? (x3): 4u7, symbol C
- added C?: 1m, symbol C
- added C?: 2.2n, symbol C
- added D?: 1N5819, symbol DIODESCH
- added K?: servo, symbol CONN_3
- added L?: INDUCTOR, symbol INDUCTOR
- added P?: dist, symbol CONN_4
- added P?: speaker, symbol CONN_2
- added P?: p1, ~, symbol CONN_CLS_28
- added P?: p2, ~, symbol CONN_CLS_28
- added P?: p3, symbol CONN_6
- added Q? (x3): PNP, ~, symbol PNP
- added Q? (x2): NPN, ~, symbol NPN
- added R?: 0, ~, symbol R
- added R? (x5): 1k, ~, symbol R
- added R?: 100, ~, symbol R
- added R?: 20k, symbol R
- added R?: 12k, symbol R
- added U?: SD, symbol SD
- added U?: 3310-LCD, symbol 3310-LCD
- added U?: NCP3063, symbol NCP3063
Connections:
- net labels added: 5v-en, dist-echo, dist-trig, filter-vdd, lcd-clk, lcd-cs, lcd-mode, lcd-mosi, lcd-rst, pb10, pb11, pb12, pb13, pb14, pb15, sd-cs, sd-miso, sd-mosi, sd-sck, servo-pwm, snd-amp-vdd
- net labels removed: boost-out
- wire segments 187 -> 320
- no-connect marks 0 -> 2
Other:
- note added: "Because servo-vcc could \nbe less then 3.3v."
- note added: "If input is 4 AA batteries, it is 6V. 6V is too \nmuch. But of 5V is taken from boost circuit \nmosfet is needed to turn it on. It is because \nof big probable consumption."
- note added: "It is not enough for sound applications.\nBecause amplifier can provide up to 1.5W \nof sound power."
- note added: "It isn't only from discovery. It is \nalso to discovery if power circuit \nis soldered."
- note added: "No need in protective diode because here \nare capacitors inductor is supposed to take \ncurrent from. These capacitors should prevent \ntransistor burning."
- moved on the sheet: C?, D?, L?, R?, U?

Commit message: Designing circuit...
Parts:
- removed C?: 1m, symbol C
- removed R? (x2): 0, ~, symbol R
- added C?: 100n, ~, symbol C
- added C?: 54u, ~, symbol CP1
- added D?: DIODESCH, ~, symbol DIODESCH
- added K?: 1-wire, symbol CONN_3
- added P?: btn-1, symbol CONN_2
- added P?: btn-2, symbol CONN_2
- added P?: btn-3, symbol CONN_2
- added P?: btn-4, symbol CONN_2
- added P?: btn-5, symbol CONN_2
- added P?: batt, symbol CONN_2
- added Q?: bc857, ~, symbol NPN
- added Q?: MOSFET_N, ~, symbol MOSFET_N
- added Q?: bc857, ~, symbol PNP
- added Q?: bc847, ~, symbol NPN
- added R? (x2): 0, ~, symbol R
- added R?: 1, ~, symbol R
- added R? (x7): 30k, ~, symbol R
- added R? (x3): 1k, ~, symbol R
- added R?: 4k7, ~, symbol R
- added R?: 10k, ~, symbol R
- added U? (x2): AD8607_2, ~, symbol AD8607_2
- added U?: DS18S20, ~, symbol DS18S20
- added U?: MINI-USB-B, ~, symbol MINI-USB-B
- L?: value INDUCTOR -> 47uH
- Q? (x4): value NPN -> bc847
- Q? (x3): value PNP -> bc857
Connections:
- net labels added: 1w-en, 1w-rx, 1w-tx, 3v3, Boot, btn-1, btn-2, btn-3, btn-4, btn-5, gnd, nc, pa0, pa1, pa10, pa11, pa12, pa13, pa14, pa15, pa2, pa3, pa4, pa5, pa6, pa7, pa8, pa9, pb0, pb1, pb2, pb3, pb4, pb5, pb6, pb7, pb8, pb9, pc0, pc1, pc10, pc11, pc12, pc13, pc14, pc15, pc2, pc3, pc4, pc5, pc6, pc7, pc8, pc9, pd0, pd1, pd2, rst, servo-en-400mA, servo-en-60mA, vbat
- net labels removed: in-400mA, in-60mA
- wire segments 320 -> 406
Other:
- note added: "3 AA batteries. \nE.i. 4.5V."
- note added: "5V adapter \nor USB slot."
- note added: "Alternative either N-P-N or MOSFET-N."
- note removed: "If input is 4 AA batteries, it is 6V. 6V is too \nmuch. But of 5V is taken from boost circuit \nmosfet is needed to turn it on. It is because \nof big probable consumption."
- moved on the sheet: C?, D?, K?, L?, P?, Q?, R?, U?

Commit message: Making scheme.
Parts:
- added P? (x4): led, symbol CONN_2
- added Q?: bc857, ~, symbol PNP
- added Q?: bc847, ~, symbol NPN
- added R? (x2): 1k, ~, symbol R
- added R? (x4): 300, ~, symbol R
- added R?: 30k, ~, symbol R
- added R?: 10k, ~, symbol R
Connections:
- net labels added: adapter-volt, battery-volt, led-en
- wire segments 406 -> 442
- no-connect marks 2 -> 6
Other:
- note added: "Because servo-vcc could \nbe less then 3.3v if batteries \npack is very discharged."
- note added: "Power instead of VDD because LED \nvoltage drop could be more then 3.3V."
- note removed: "Because servo-vcc could \nbe less then 3.3v."
- moved on the sheet: P?, R?

Commit message: Drawing scheme.
Parts:
- removed C? (x3): 100n, ~, symbol C
- removed C? (x2): 4u7, ~, symbol C
- removed C?: 5p, ~, symbol C
- removed Q?: bc857, ~, symbol PNP
- removed Q?: MOSFET_N, ~, symbol MOSFET_N
- removed R?: 10k, ~, symbol R
- removed R?: 100k, ~, symbol R
- removed R? (x2): 30k, ~, symbol R
- removed R? (x3): 0, ~, symbol R
- removed R? (x2): 1k, ~, symbol R
- removed R?: 1, ~, symbol R
- removed U?: LM4861, ~, symbol LM4861
- removed U?: AD8607_2, ~, symbol AD8607_2
- added C?: 54u, ~, symbol CP1
- added C? (x2): 4u7, ~, symbol C
- added C?: 100n, ~, symbol C
- added Q? (x2): bc847, ~, symbol NPN
- added Q? (x2): bc857, ~, symbol PNP
- added R? (x2): 0, ~, symbol R
- added R? (x6): 1k, ~, symbol R
- added R?: 5k1, ~, symbol R
- added R?: 10k, ~, symbol R
- L?: value INDUCTOR -> 47uH
- Q?: value bc857 -> bc847
Connections:
- net labels removed: snd-amp-vdd
- wire segments 442 -> 422
Other:
- note added: "This resistances ratio \nconverts 3.3V to 5V range."
- note removed: "Alternative either N-P-N or MOSFET-N."
- moved on the sheet: C?, D?, K?, P?, Q?, R?, U?, U?A, U?B
