File: electric/scheme-proto/clock-proto.kicad_pcb (KiCad board)
At the start: 2 copper layers, 60.5 x 88.5 mm, 123 parts, among them K1 servo, K2 1-wire, P1 batt, P10 led, P11 p2, P12 btn-4, P13 led, P14 led, P15 btn-5, P2 speaker, P3 dist, P4 btn-1, P5 btn-2, P6 btn-3, P7 led, P8 p1, P9 p3, Q1 bc857, Q10 bc857, Q11 bc847, Q12 bc857, Q13 bc847, Q15 bc847, Q16 bc847, Q17 bc857, Q18 bc857, Q2 bc847, Q3 bc857, Q4 bc847, Q5 irlml2244, Q6 bc847, Q7 bc857, Q8 bc847, Q9 bc857, U1 3310-LCD, U2 AD8607_2, U3 SD, U4 MINI-USB-B, U6 NCP3063, U7 NCP3063, U8 DS18S20

Commit message: Recalculated values for 12kHz low pass filter.
Parts:
- C6: value 4n -> 8.2n
- C7: value 1n -> 1.2n
- C8: value 68n -> 15n
- C9: value 1n -> 100p
- R10: value 10k -> 12k
- R13: value 20k -> 5k1
- R16: value 2k7 -> 4k7
- R17: value 1k3 -> 15k
- R18: value 2k7 -> 5k6
- R19: value 15k -> 12k
- R9: value 20k -> 4k3
Changed lines of the file:
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@@
     (links 236)
     (no_connects 0)
-    (area 119.449999 60.449999 180.050001 149.050001)
+    (area 119.449999 58.01106 180.050001 149.050001)
     (thickness 1.6)
     (drawings 10)
@@
   )
   (setup
-    (last_trace_width 0.4)
+    (last_trace_width 0.254)
     (user_trace_width 0.4)
     (user_trace_width 0.6)
@@
       (effects (font (size 0.50038 0.50038) (thickness 0.10922)))
     )
-    (fp_text value 20k (at 0 0.381 270) (layer F.SilkS)
+    (fp_text value 4k3 (at 0 0.381 270) (layer F.SilkS)
       (effects (font (size 0.50038 0.50038) (thickness 0.10922)))
     )
@@
       (effects (font (size 0.50038 0.50038) (thickness 0.10922)))
     )
-    (fp_text value 2k7 (at 0 0.381 270) (layer F.SilkS)
+    (fp_text value 5k6 (at 0 0.381 270) (layer F.SilkS)
       (effects (font (size 0.50038 0.50038) (thickness 0.10922)))
     )
@@
       (effects (font (size 0.50038 0.50038) (thickness 0.10922)))
     )
-    (fp_text value 15k (at 0 0.381 270) (layer F.SilkS)
+    (fp_text value 12k (at 0 0.381 270) (layer F.SilkS)
       (effects (font (size 0.50038 0.50038) (thickness 0.10922)))
     )
@@
       (effects (font (size 0.50038 0.50038) (thickness 0.10922)))
     )
-    (fp_text value 10k (at 0 0.381 180) (layer F.SilkS)
+    (fp_text value 12k (at 0 0.381 180) (layer F.SilkS)
       (effects (font (size 0.50038 0.50038) (thickness 0.10922)))
     )
@@
       (effects (font (size 0.50038 0.50038) (thickness 0.10922)))
     )
-    (fp_text value 1n (at 0 0.381 270) (layer F.SilkS)
+    (fp_text value 100p (at 0 0.381 270) (layer F.SilkS)
       (effects (font (size 0.50038 0.50038) (thickness 0.10922)))
     )
@@
       (effects (font (size 0.50038 0.50038) (thickness 0.10922)))
     )
-    (fp_text value 68n (at 0 0.381 90) (layer F.SilkS)
+    (fp_text value 15n (at 0 0.381 90) (layer F.SilkS)
       (effects (font (size 0.50038 0.50038) (thickness 0.10922)))
     )
@@
       (effects (font (size 0.50038 0.50038) (thickness 0.10922)))
     )
-    (fp_text value 2k7 (at 0 0.381 270) (layer F.SilkS)
+    (fp_text value 4k7 (at 0 0.381 270) (layer F.SilkS)
       (effects (font (size 0.50038 0.50038) (thickness 0.10922)))
     )
@@
       (effects (font (size 0.50038 0.50038) (thickness 0.10922)))
     )
-    (fp_text value 1k3 (at 0 0.381) (layer F.SilkS)
+    (fp_text value 15k (at 0 0.381) (layer F.SilkS)
       (effects (font (size 0.50038 0.50038) (thickness 0.10922)))
     )
@@
       (effects (font (size 0.50038 0.50038) (thickness 0.10922)))
     )
-    (fp_text value 20k (at 0 0.381 270) (layer F.SilkS)
+    (fp_text value 5k1 (at 0 0.381 270) (layer F.SilkS)
       (effects (font (size 0.50038 0.50038) (thickness 0.10922)))
     )
@@
       (effects (font (size 0.50038 0.50038) (thickness 0.10922)))
     )
-    (fp_text value 1n (at 0 0.381 270) (layer F.SilkS)
+    (fp_text value 1.2n (at 0 0.381 270) (layer F.SilkS)
       (effects (font (size 0.50038 0.50038) (thickness 0.10922)))
     )
@@
       (effects (font (size 0.50038 0.50038) (thickness 0.10922)))
     )
-    (fp_text value 4n (at 0 0.381 180) (layer F.SilkS)
+    (fp_text value 8.2n (at 0 0.381 180) (layer F.SilkS)
       (effects (font (size 0.50038 0.50038) (thickness 0.10922)))
     )
@@
   (segment (start 176.3776 95.504) (end 176.3776 93.5736) (width 0.4) (layer F.Cu) (net 40))
   (segment (start 175.9331 95.9485) (end 176.3776 95.504) (width 0.4) (layer F.Cu) (net 40))
-  (segment (start 173.05 143.3525) (end 173.05 144.89) (width 0.4) (layer F.Cu) (net 41) (status C00000))
-  (segment (start 173.05 144.89) (end 173.1 144.94) (width 0.4) (layer F.Cu) (net 41) (status C00000))
+  (segment (start 173.05 143.3525) (end 173.05 144.89) (width 0.4) (layer F.Cu) (net 41))
+  (segment (start 173.05 144.89) (end 173.1 144.94) (width 0.4) (layer F.Cu) (net 41))
   (segment (start 173.1 144.94) (end 173.16 144.94) (width 0.4) (layer F.Cu) (net 41))
   (segment (start 175.05 143.05) (end 176.91 143.05) (width 0.4) (layer F.Cu) (net 41))
@@
   (segment (start 127.9144 117.6909) (end 129.8448 117.6909) (width 0.4) (layer F.Cu) (net 67))
   (segment (start 129.8448 117.6909) (end 130.302 118.1481) (width 0.4) (layer F.Cu) (net 67))
-  (segment (start 173.05 141.4475) (end 173.05 139.91) (width 0.4) (layer F.Cu) (net 68) (status C00000))
-  (segment (start 173.05 139.91) (end 173.1 139.86) (width 0.4) (layer F.Cu) (net 68) (status C00000))
+  (segment (start 173.05 141.4475) (end 173.05 139.91) (width 0.4) (layer F.Cu) (net 68))
+  (segment (start 173.05 139.91) (end 173.1 139.86) (width 0.4) (layer F.Cu) (net 68))
   (segment (start 161.2 134.8) (end 161.25 134.8) (width 0.4) (layer F.Cu) (net 68))
   (segment (start 161.25 134.8) (end 166.31 139.86) (width 0.4) (layer F.Cu) (net 68))
